File: _autosave-micromouse_01-2.kicad_sch (KiCad schematic)
At the start: 64 parts, among them IC6 PCA9632TK,118, J1 Conn_01x02_Pin, M3 Fan_Motor, Q1 MCM3400A-TP, Q2 MCM3400A-TP, Q3 MCM3400A-TP, Q4 Q_PMOS_GSD, Q5 Q_PMOS_GSD, Q6 Q_PMOS_GSD, SW3 SSSS810701, U1 SMT-0440-S-R, U2 LBR-127HLD, U3 LBR-127HLD, U4 LBR-127HLD, U5 LBR-127HLD, U6 LXDC55FAAA-203, U7 MCP73831-2-OT, U8 WS2812-2020

Commit message: 仮変更
Parts:
- removed D12: 1N4148W, Diode_SMD:D_SOD-123, symbol Diode:1N4148W
- removed D7: 1N5819HW-7-F, footprints:SOD3715X145N, symbol 1N5819HW-7-F:1N5819HW-7-F
- added D5, D7: CCS15S40,L3F, footprints:SOD-963 CST2C_TOS, symbol Diode:1N4148W
- R24, R27: value R -> 47k
Connections:
- net VBUS: now also D5.2 (A), D7.2 (A)
- net at Q5.2 (S), Q6.2 (S), R27.1: now also D7.1 (K)
- net at Q4.1 (G), Q5.1 (G), R24.1: now also D5.1 (K)
Changed lines of the file:
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@@
-    (stroke (width 0) (type default))
-  )
-  (wire (pts (xy 233.68 116.84) (xy 233.68 137.16))
     (stroke (width 0) (type default))
   )
@@
     (stroke (width 0) (type default))
   )
-  (wire (pts (xy 210.82 139.7) (xy 210.82 162.56))
-    (stroke (width 0) (type default))
-  )
   (wire (pts (xy 144.78 54.61) (xy 144.78 87.63))
     (stroke (width 0) (type default))
@@
     (stroke (width 0) (type default))
   )
+  (wire (pts (xy 233.68 146.05) (xy 233.68 162.56))
+    (stroke (width 0) (type default))
+  )
   (wire (pts (xy 102.87 139.7) (xy 102.87 143.51))
     (stroke (width 0) (type default))
@@
     (stroke (width 0) (type default))
   )
+  (wire (pts (xy 210.82 140.97) (xy 210.82 162.56))
+    (stroke (width 0) (type default))
+  )
   (wire (pts (xy 86.36 102.87) (xy 92.71 102.87))
     (stroke (width 0) (type default))
@@
     (stroke (width 0) (type default))
   )
-  (wire (pts (xy 233.68 147.32) (xy 233.68 162.56))
-    (stroke (width 0) (type default))
-  )
   (wire (pts (xy 99.06 87.63) (xy 116.84 87.63))
     (stroke (width 0) (type default))
@@
     (stroke (width 0) (type default))
   )
-  (wire (pts (xy 210.82 127) (xy 210.82 132.08))
+  (wire (pts (xy 210.82 127) (xy 210.82 133.35))
     (stroke (width 0) (type default))
   )
@@
   )
   (wire (pts (xy 194.31 93.98) (xy 209.55 93.98))
+    (stroke (width 0) (type default))
+  )
+  (wire (pts (xy 233.68 116.84) (xy 233.68 138.43))
     (stroke (width 0) (type default))
   )
@@
     (property "Intersheetrefs" "${INTERSHEET_REFS}" (at 74.93 70.4934 90)
       (effects (font (size 1.27 1.27)) (justify left) hide)
+    )
+  )
+  (symbol (lib_id "Diode:1N4148W") (at 210.82 137.16 270) (unit 1)
+    (in_bom yes) (on_board yes) (dnp no)
+    (property "Reference" "D5" (at 213.36 134.62 90)
+      (effects (font (size 1.27 1.27)) (justify left))
+    )
+    (property "Value" "CCS15S40,L3F" (at 208.28 132.08 0)
+      (effects (font (size 1.27 1.27)) (justify left))
+    )
+    (property "Footprint" "footprints:SOD-963   CST2C_TOS" (at 206.375 137.16 0)
+      (effects (font (size 1.27 1.27)) hide)
+    )
+    (property "Datasheet" "https://www.vishay.com/docs/85748/1n4148w.pdf" (at 210.82 137.16 0)
+      (effects (font (size 1.27 1.27)) hide)
+    )
+    (property "Sim.Device" "D" (at 210.82 137.16 0)
+      (effects (font (size 1.27 1.27)) hide)
+    )
+    (property "Sim.Pins" "1=K 2=A" (at 210.82 137.16 0)
+      (effects (font (size 1.27 1.27)) hide)
+    )
+    (pin "1")
+    (pin "2")
+    (instances
+      (project "micromouse_01_cp2"
+        (path "/619a00a9-cfa2-4255-85f4-bd5efe9f55d3/d924c110-d411-42e8-bf64-5ff34a3957e3"
+          (reference "D5") (unit 1)
+        )
+      )
     )
   )
@@
     )
   )
-  (symbol (lib_id "1N5819HW-7-F:1N5819HW-7-F") (at 233.68 142.24 90) (unit 1)
-    (in_bom yes) (on_board yes) (dnp no) (fields_autoplaced)
-    (property "Reference" "D7" (at 236.22 140.97 90)
-      (effects (font (size 1.27 1.27)) (justify right))
-    )
-    (property "Value" "1N5819HW-7-F" (at 236.22 143.51 90)
-      (effects (font (size 1.27 1.27)) (justify right))
-    )
-    (property "Footprint" "footprints:SOD3715X145N" (at 233.68 142.24 0)
-      (effects (font (size 1.27 1.27)) (justify bottom) hide)
-    )
-    (property "Datasheet" "" (at 233.68 142.24 0)
-      (effects (font (size 1.27 1.27)) hide)
-    )
-    (property "PARTREV" "18-2" (at 233.68 142.24 0)
-      (effects (font (size 1.27 1.27)) (justify bottom) hide)
-    )
-    (property "STANDARD" "IPC-7351B" (at 233.68 142.24 0)
-      (effects (font (size 1.27 1.27)) (justify bottom) hide)
-    )
-    (property "MANUFACTURER" "Diodes Inc." (at 233.68 142.24 0)
-      (effects (font (size 1.27 1.27)) (justify bottom) hide)
-    )
-    (pin "A")
-    (pin "C")
-    (instances
-      (project "micromouse_01_cp2"
-        (path "/619a00a9-cfa2-4255-85f4-bd5efe9f55d3/d924c110-d411-42e8-bf64-5ff34a3957e3"
-          (reference "D7") (unit 1)
-        )
-      )
-    )
-  )
   (symbol (lib_id "power:GND") (at 270.51 35.56 0) (mirror y) (unit 1)
     (in_bom yes) (on_board yes) (dnp no) (fields_autoplaced)
@@
       (effects (font (size 1.27 1.27)) (justify left))
     )
-    (property "Value" "R" (at 246.38 125.73 0)
+    (property "Value" "47k" (at 246.38 125.73 0)
       (effects (font (size 1.27 1.27)) (justify left))
     )
@@
         (path "/619a00a9-cfa2-4255-85f4-bd5efe9f55d3/d924c110-d411-42e8-bf64-5ff34a3957e3"
           (reference "R30") (unit 1)
-        )
-      )
-    )
-  )
-  (symbol (lib_id "Diode:1N4148W") (at 210.82 135.89 270) (unit 1)
-    (in_bom yes) (on_board yes) (dnp no) (fields_autoplaced)
-    (property "Reference" "D12" (at 213.36 134.62 90)
-      (effects (font (size 1.27 1.27)) (justify left))
-    )
-    (property "Value" "1N4148W" (at 213.36 137.16 90)
-      (effects (font (size 1.27 1.27)) (justify left))
-    )
-    (property "Footprint" "Diode_SMD:D_SOD-123" (at 206.375 135.89 0)
-      (effects (font (size 1.27 1.27)) hide)
-    )
-    (property "Datasheet" "https://www.vishay.com/docs/85748/1n4148w.pdf" (at 210.82 135.89 0)
-      (effects (font (size 1.27 1.27)) hide)
-    )
-    (property "Sim.Device" "D" (at 210.82 135.89 0)
-      (effects (font (size 1.27 1.27)) hide)
-    )
-    (property "Sim.Pins" "1=K 2=A" (at 210.82 135.89 0)
-      (effects (font (size 1.27 1.27)) hide)
-    )
-    (pin "1")
-    (pin "2")
-    (instances
-      (project "micromouse_01_cp2"
-        (path "/619a00a9-cfa2-4255-85f4-bd5efe9f55d3/d924c110-d411-42e8-bf64-5ff34a3957e3"
-          (reference "D12") (unit 1)
         )
       )
@@
       (effects (font (size 1.27 1.27)) (justify left))
     )
-    (property "Value" "R" (at 223.52 143.51 0)
+    (property "Value" "47k" (at 223.52 143.51 0)
       (effects (font (size 1.27 1.27)) (justify left))
     )
@@
         )
       )
+    )
+  )
+  (symbol (lib_id "Diode:1N4148W") (at 233.68 142.24 270) (unit 1)
+    (in_bom yes) (on_board yes) (dnp no)
+    (property "Reference" "D7" (at 236.22 139.7 90)
+      (effects (font (size 1.27 1.27)) (justify left))
+    )
+    (property "Value" "CCS15S40,L3F" (at 231.14 137.16 0)
+      (effects (font (size 1.27 1.27)) (justify left))
+    )
+    (property "Footprint" "footprints:SOD-963   CST2C_TOS" (at 229.235 142.24 0)
+      (effects (font (size 1.27 1.27)) hide)
+    )
+    (property "Datasheet" "https://www.vishay.com/docs/85748/1n4148w.pdf" (at 233.68 142.24 0)
+      (effects (font (size 1.27 1.27)) hide)
+    )
+    (property "Sim.Device" "D" (at 233.68 142.24 0)
+      (effects (font (size 1.27 1.27)) hide)
+    )
+    (property "Sim.Pins" "1=K 2=A" (at 233.68 142.24 0)
+      (effects (font (size 1.27 1.27)) hide)
+    )
+    (pin "1")
+    (pin "2")
+    (instances
+      (project "micromouse_01_cp2"
+        (path "/619a00a9-cfa2-4255-85f4-bd5efe9f55d3/d924c110-d411-42e8-bf64-5ff34a3957e3"
+          (reference "D7") (unit 1)
+        )
+      )
